File: hardware/pcb/kxusbc2_chg.kicad_sch (KiCad schematic)
At the start: 49 parts, among them Q1 CSD17581Q3A, Q2 CSD17581Q3A, Q3 CSD17581Q3A, Q4 CSD17581Q3A, U1 BQ25792RQMR

Commit message: Implement DC jack reverse polarity protection using P-channel MOSFET (closes #6)
Parts:
- removed TP1: SYS, TestPoint:TestPoint_Pad_2.5x2.5mm, symbol Connector:TestPoint
- added D10: 5.6V, Diode_SMD:D_SOD-523, symbol Device:D_Zener
- added Q5: CSD25402Q3A, VSON-8_TI_CSD:VSON-8_3.3x3.3mm_TI_CSD, symbol Transistor_FET:CSD25402Q3A
- added R12: 100k, Resistor_SMD:R_0402_1005Metric, symbol Device:R
- C12: footprint Capacitor_SMD:C_0603_1608Metric_Pad1.08x0.95mm_HandSolder -> Capacitor_SMD:C_0402_1005Metric
- C3, C4: footprint Capacitor_SMD:C_0603_1608Metric_Pad1.08x0.95mm_HandSolder -> Capacitor_SMD:C_0603_1608Metric
- Q1, Q2, Q3, Q4: footprint VSON-8_csd17581q3a:VSON-8_csd17581q3a -> VSON-8_TI_CSD:VSON-8_3.3x3.3mm_TI_CSD
- R1: footprint Resistor_SMD:R_0603_1608Metric_Pad0.98x0.95mm_HandSolder -> Resistor_SMD:R_0402_1005Metric
- renumbered TP2 to TP1, TP3 to TP2, TP4 to TP3
Connections:
- net GND: now also R12.2
- net VDC: now also Q5.1 (D), Q5.2 (D), Q5.3 (D); no longer C22.1, Q3.5 (D), R11.1, U1.8 (VAC2)
- new net: D10.2 (A), Q5.4 (G), R12.1
- new net VDC_SAFE: C22.1, D10.1 (K), Q3.5 (D), Q5.5 (S), R11.1, U1.8 (VAC2)
Other:
- moved on the sheet: C1, C10, C12, C13, C14, C17, C18, C19, C2, C20, C21, C22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
