File: hardware/pcb/kxusbc2.kicad_sch (KiCad schematic)
At the start: 7 parts, among them J1 Conn_01x03, J3 Conn_01x03, J4 Conn_01x03, J7 Conn_01x01, J8 Conn_01x01

Commit message: Add test points for I2C and interrupt lines
Parts:
- added TP4, TP5, TP6, TP7: TestPoint, TestPoint:TestPoint_Pad_D1.0mm, symbol Connector:TestPoint
Connections:
- net Charger/SCL: now also TP4.1
- net Charger/SDA: now also TP5.1
- net Charger/~{BQ_INT}: now also TP7.1
- net USB-C/~{FUSB_INT}: now also TP6.1

Commit message: Add JLCPCB project DB (for rotation corrections), exclude test points from BOM
Parts:
- TP4, TP5, TP6, TP7: now left out of the parts list
Changed lines of the file:
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@@
 		(unit 1)
 		(exclude_from_sim no)
-		(in_bom yes)
+		(in_bom no)
 		(on_board yes)
 		(dnp no)
@@
 		(unit 1)
 		(exclude_from_sim no)
-		(in_bom yes)
+		(in_bom no)
 		(on_board yes)
 		(dnp no)
@@
 		(unit 1)
 		(exclude_from_sim no)
-		(in_bom yes)
+		(in_bom no)
 		(on_board yes)
 		(dnp no)
@@
 		(unit 1)
 		(exclude_from_sim no)
-		(in_bom yes)
-		(on_board yes)
-		(dnp no)
+		(in_bom no)
+		(on_board yes)
+		(dnp no)

Commit message: Update legend, DNP
Other:
- note added: "KX2 interface"
Changed lines of the file:
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@@
 		(title "KXUSBC2 – Internal USB-C charger for the Elecraft KX2")
 		(comment 1 "Licensed under CERN-OHL-W v2")
-		(comment 2 "© 2025 HB9DQM")
+		(comment 2 "© 2025-2026 HB9DQM")
+	)
+	(text "KX2 interface"
+		(exclude_from_sim no)
+		(at 224.028 71.882 90)
+		(effects
+			(font
+				(size 2.54 2.54)
+			)
+		)
 	)
 	(junction
