File: hardware/pcb/kxusbc2_uc.kicad_sch (KiCad schematic)
At the start: 19 parts, among them J2 UPDI, J6 Serial, SW1 SW_Push, U2 ATtiny3226-M, U4 RT9058-33GV, U5 LP5815DRLR, Y1 32.768 kHz

Commit message: Make debug/serial pads more staggered (closes #18)
Parts:
- J2, J6: now not fitted
Changed lines of the file:
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@@
 		(in_bom no)
 		(on_board yes)
-		(dnp no)
+		(dnp yes)
 		(property "Reference" "J2"
 			(at 137.922 44.5078 0)
@@
 		(in_bom no)
 		(on_board yes)
-		(dnp no)
+		(dnp yes)
 		(property "Reference" "J6"
 			(at 163.322 76.1422 0)
