File: hardware/pcb/kxusbc2_uc.kicad_sch (KiCad schematic)
At the start: 21 parts, among them J2 UPDI, J6 Serial, SW1 SW_Push, U2 ATtiny3226-M, U4 RT9058-33GV, U5 LP5815DRLR, Y1 32.768 kHz

Commit message: Fix RGB LED pin order
Parts:
- D1: symbol LED:APFA3010 -> Device:LED_RGBA
Connections:
- net +3V3: now also D1.4 (A); no longer D1.2 (A)
- net at U5.6 (OUT2): now also D1.1 (RK); no longer D1.3 (G)
- net at U5.7 (OUT1): now also D1.2 (GK); no longer D1.4 (B)
- net at U5.8 (OUT0): now also D1.3 (BK); no longer D1.1 (R)
Changed lines of the file:
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@@
 	(wire
 		(pts
-			(xy 208.28 148.59) (xy 205.74 148.59)
+			(xy 203.2 153.67) (xy 208.28 153.67)
 		)
 		(stroke
@@
 	(wire
 		(pts
-			(xy 205.74 147.32) (xy 194.31 147.32)
-		)
-		(stroke
-			(width 0)
-			(type default)
-		)
-	)
-	(wire
-		(pts
 			(xy 184.15 91.44) (xy 177.8 91.44)
 		)
@@
 	(wire
 		(pts
-			(xy 203.2 153.67) (xy 208.28 153.67)
-		)
-		(stroke
-			(width 0)
-			(type default)
-		)
-	)
-	(wire
-		(pts
 			(xy 163.83 82.55) (xy 163.83 85.09)
 		)
@@
 	(wire
 		(pts
+			(xy 203.2 152.4) (xy 203.2 153.67)
+		)
+		(stroke
+			(width 0)
+			(type default)
+		)
+	)
+	(wire
+		(pts
 			(xy 114.3 85.09) (xy 118.11 85.09)
 		)
@@
 	(wire
 		(pts
-			(xy 200.66 143.51) (xy 208.28 143.51)
+			(xy 203.2 147.32) (xy 203.2 143.51)
 		)
 		(stroke
@@
 	(wire
 		(pts
-			(xy 205.74 148.59) (xy 205.74 147.32)
-		)
-		(stroke
-			(width 0)
-			(type default)
-		)
-	)
-	(wire
-		(pts
 			(xy 139.7 118.11) (xy 139.7 119.38)
 		)
@@
 	(wire
 		(pts
-			(xy 203.2 149.86) (xy 203.2 153.67)
+			(xy 215.9 46.99) (xy 218.44 46.99)
 		)
 		(stroke
@@
 	(wire
 		(pts
-			(xy 215.9 46.99) (xy 218.44 46.99)
+			(xy 146.05 62.23) (xy 177.8 62.23)
 		)
 		(stroke
@@
 	(wire
 		(pts
-			(xy 146.05 62.23) (xy 177.8 62.23)
+			(xy 194.31 78.74) (xy 194.31 80.01)
 		)
 		(stroke
@@
 	(wire
 		(pts
-			(xy 194.31 78.74) (xy 194.31 80.01)
+			(xy 156.21 152.4) (xy 166.37 152.4)
 		)
 		(stroke
@@
 	(wire
 		(pts
-			(xy 156.21 152.4) (xy 166.37 152.4)
+			(xy 203.2 143.51) (xy 208.28 143.51)
 		)
 		(stroke
@@
 	(wire
 		(pts
+			(xy 203.2 149.86) (xy 203.2 148.59)
+		)
+		(stroke
+			(width 0)
+			(type default)
+		)
+	)
+	(wire
+		(pts
 			(xy 218.44 39.37) (xy 227.33 39.37)
 		)
@@
 	(wire
 		(pts
+			(xy 203.2 148.59) (xy 208.28 148.59)
+		)
+		(stroke
+			(width 0)
+			(type default)
+		)
+	)
+	(wire
+		(pts
 			(xy 129.54 106.68) (xy 135.89 106.68)
 		)
@@
 	(wire
 		(pts
-			(xy 152.4 152.4) (xy 156.21 152.4)
+			(xy 194.31 147.32) (xy 203.2 147.32)
 		)
 		(stroke
@@
 	(wire
 		(pts
-			(xy 240.03 67.31) (xy 251.46 67.31)
+			(xy 152.4 152.4) (xy 156.21 152.4)
 		)
 		(stroke
@@
 	(wire
 		(pts
-			(xy 160.02 149.86) (xy 160.02 161.29)
+			(xy 240.03 67.31) (xy 251.46 67.31)
 		)
 		(stroke
@@
 	(wire
 		(pts
-			(xy 114.3 95.25) (xy 137.16 95.25)
+			(xy 160.02 149.86) (xy 160.02 161.29)
 		)
 		(stroke
@@
 	(wire
 		(pts
-			(xy 194.31 144.78) (xy 195.58 144.78)
+			(xy 114.3 95.25) (xy 137.16 95.25)
 		)
 		(stroke
@@
 	(wire
 		(pts
-			(xy 80.01 100.33) (xy 83.82 100.33)
+			(xy 194.31 144.78) (xy 195.58 144.78)
 		)
 		(stroke
@@
 	(wire
 		(pts
-			(xy 200.66 152.4) (xy 200.66 143.51)
+			(xy 80.01 100.33) (xy 83.82 100.33)
 		)
 		(stroke
@@
 	(wire
 		(pts
-			(xy 194.31 152.4) (xy 200.66 152.4)
+			(xy 152.4 161.29) (xy 160.02 161.29)
 		)
 		(stroke
@@
 	(wire
 		(pts
-			(xy 152.4 161.29) (xy 160.02 161.29)
+			(xy 195.58 161.29) (xy 160.02 161.29)
 		)
 		(stroke
@@
 	(wire
 		(pts
-			(xy 195.58 161.29) (xy 160.02 161.29)
+			(xy 73.66 72.39) (xy 73.66 73.66)
 		)
 		(stroke
@@
 	(wire
 		(pts
-			(xy 73.66 72.39) (xy 73.66 73.66)
+			(xy 129.54 118.11) (xy 139.7 118.11)
 		)
 		(stroke
@@
 	(wire
 		(pts
-			(xy 129.54 118.11) (xy 139.7 118.11)
+			(xy 116.84 72.39) (xy 114.3 72.39)
 		)
 		(stroke
@@
 	(wire
 		(pts
-			(xy 116.84 72.39) (xy 114.3 72.39)
+			(xy 194.31 152.4) (xy 203.2 152.4)
 		)
 		(stroke
@@
 	)
 	(symbol
-		(lib_id "LED:APFA3010")
+		(lib_id "Device:LED_RGBA")
 		(at 213.36 148.59 0)
 		(unit 1)
@@
 		(fields_autoplaced yes)
 		(property "Reference" "D1"
-			(at 213.36 135.5555 0)
+			(at 213.36 136.0635 0)
 			(effects
 				(font
@@
 		)
 		(property "Value" "LTST-C19HE1WT-H"
-			(at 213.36 137.9798 0)
+			(at 213.36 138.4878 0)
 			(effects
 				(font
@@
 		)
 		(property "Footprint" "LED_SMD:LED_LiteOn_LTST-C19HE1WT"
-			(at 213.36 135.89 0)
+			(at 213.36 149.86 0)
 			(effects
 				(font
@@
 			)
 		)
-		(property "Datasheet" "http://www.kingbrightusa.com/images/catalog/SPEC/APFA3010LSEEZGKQBKC.pdf"
-			(at 213.36 160.02 0)
+		(property "Datasheet" "~"
+			(at 213.36 149.86 0)
 			(effects
 				(font
@@
 			)
 		)
-		(property "Description" "LED RGB, Common Anode, SMD, 3.0x1.5mm, Horizontal"
+		(property "Description" "RGB LED, red/green/blue/anode"
 			(at 213.36 148.59 0)
 			(effects
