File: hardware/pcb/kxusbc2_uc.kicad_sch (KiCad schematic)
At the start: 21 parts, among them J2 UPDI, J6 Serial, SW1 SW_Push, U2 ATtiny3226-M, U4 RT9058-33GV, U5 LP5815DRLR, Y1 32.768 kHz

Commit message: Switch back to right-angle LED without light pipe (closes #41)
Parts:
- D1: value LTST-C19HE1WT-H -> APFA3010LSEEZGKQBKC; footprint LED_SMD:LED_LiteOn_LTST-C19HE1WT -> LED_SMD:LED_Kingbright_APFA3010_3x1.5mm_Horizontal; symbol Device:LED_RGBA -> LED:APFA3010; LCSC C427425 -> C5393554
Connections:
- net +3V3: now also D1.2 (A); no longer D1.4 (A)
- net at U5.7 (OUT1): now also D1.3 (G); no longer D1.2 (GK)
- net at U5.8 (OUT0): now also D1.4 (B); no longer D1.3 (BK)
Changed lines of the file:
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@@
 	)
 	(symbol
-		(lib_id "Device:LED_RGBA")
+		(lib_id "LED:APFA3010")
 		(at 213.36 148.59 0)
 		(unit 1)
@@
 		(fields_autoplaced yes)
 		(property "Reference" "D1"
-			(at 213.36 136.0635 0)
+			(at 213.36 135.5555 0)
 			(effects
 				(font
@@
 			)
 		)
-		(property "Value" "LTST-C19HE1WT-H"
-			(at 213.36 138.4878 0)
+		(property "Value" "APFA3010LSEEZGKQBKC"
+			(at 213.36 137.9798 0)
 			(effects
 				(font
@@
 			)
 		)
-		(property "Footprint" "LED_SMD:LED_LiteOn_LTST-C19HE1WT"
-			(at 213.36 149.86 0)
+		(property "Footprint" "LED_SMD:LED_Kingbright_APFA3010_3x1.5mm_Horizontal"
+			(at 213.36 135.89 0)
 			(effects
 				(font
@@
 			)
 		)
-		(property "Datasheet" "~"
-			(at 213.36 149.86 0)
+		(property "Datasheet" "http://www.kingbrightusa.com/images/catalog/SPEC/APFA3010LSEEZGKQBKC.pdf"
+			(at 213.36 160.02 0)
 			(effects
 				(font
@@
 			)
 		)
-		(property "Description" "RGB LED, red/green/blue/anode"
+		(property "Description" "LED RGB, Common Anode, SMD, 3.0x1.5mm, Horizontal"
 			(at 213.36 148.59 0)
 			(effects
@@
 			)
 		)
-		(property "LCSC" "C427425"
+		(property "LCSC" "C5393554"
 			(at 213.36 148.59 0)
 			(effects

Commit message: Update legend, DNP
Parts:
- J2, J6: now fitted
Changed lines of the file:
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@@
 		(title "Microcontroller and LED")
 		(comment 1 "Licensed under CERN-OHL-W v2")
-		(comment 2 "© 2025 HB9DQM")
+		(comment 2 "© 2025-2026 HB9DQM")
 	)
 	(rectangle
@@
 		(in_bom no)
 		(on_board yes)
-		(dnp yes)
+		(dnp no)
 		(property "Reference" "J2"
 			(at 137.922 44.5078 0)
@@
 		(in_bom no)
 		(on_board yes)
-		(dnp yes)
+		(dnp no)
 		(property "Reference" "J6"
 			(at 163.322 76.1422 0)

Commit message: Increase crystal load capacitors to 22p for more precise frequency pre-calibration
Parts:
- C32, C33: value 18p -> 22p; LCSC C1549 -> C1555
Changed lines of the file:
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@@
 			)
 		)
-		(property "Value" "18p"
+		(property "Value" "22p"
 			(at 126.619 114.2421 0)
 			(effects
@@
 			)
 		)
-		(property "LCSC" "C1549"
+		(property "LCSC" "C1555"
 			(at 129.54 113.03 0)
 			(effects
@@
 			)
 		)
-		(property "Value" "18p"
+		(property "Value" "22p"
 			(at 152.781 114.2421 0)
 			(effects
@@
 			)
 		)
-		(property "LCSC" "C1549"
+		(property "LCSC" "C1555"
 			(at 149.86 113.03 0)
 			(effects
