File: hardware/pcb/kxusbc2.kicad_pcb (KiCad board)
At the start: 4 copper layers, 69 x 19.2 mm, 95 parts, among them J1 Conn_01x03, J2 UPDI, J3 Conn_01x03, J4 Conn_01x03, J5 GT-USB-7055AB, J6 Serial, J7 Conn_01x01, J8 Conn_01x01, Q1 CSD17581Q3A, Q2 CSD17581Q3A, Q3 CSD17581Q3A, Q4 CSD17581Q3A, Q5 CSD25402Q3A, SW1 SW_Push, U1 BQ25792RQMR, U2 ATtiny3226-M, U3 TLV9301xDCK, U4 RT9058-33GV, U5 LP5815DRLR, U7 FUSB302BMPX, Y1 32.768 kHz

Commit message: Add test points for I2C and interrupt lines
Parts:
- added TP4: TestPoint, TestPoint:TestPoint_Pad_D1.0mm, B.Cu at (153.8, 115.7)
- added TP5: TestPoint, TestPoint:TestPoint_Pad_D1.0mm, B.Cu at (152.5, 121.2)
- added TP6: TestPoint, TestPoint:TestPoint_Pad_D1.0mm, B.Cu at (121.4, 118.2)
- added TP7: TestPoint, TestPoint:TestPoint_Pad_D1.0mm, B.Cu at (124.3, 111.5)
Routing:
- net /USB-C/~{FUSB_INT}: track 13.9 -> 15.3 mm
- net /Charger/SDA: track 80.6 -> 81.9 mm
- net /Charger/SCL: track 90.3 -> 91.5 mm
- net /Charger/~{BQ_INT}: track 30.4 -> 31.3 mm

Commit message: Reduce PCB height by 0.2 mm to improve fit (screws), and make U-shaped cutout for RF PCB screw 0.3 mm deeper (#45)
Parts:
- moved C39 2.12 mm to (122.9, 122.8)
Routing:
- net GND: track 8.98 -> 11.3 mm, vias 147 -> 141
- net /Charger/VBUS: track 104.1 -> 104.6 mm
- net /Battery monitor/12VSW: vias 2 -> 4
Other:
- board size 69 x 19.2 mm -> 69 x 19 mm
- board text added: "rev3"
- board text added: "© HB9DQM 2026"
- board text removed: "rev2"
- board text removed: "© HB9DQM 2025"

Commit message: Switch back to right-angle LED without light pipe (closes #41)
Parts:
- removed LPI: Lightpipe_Bivar_SLP3-150-100-F, OptoDevice:Lightpipe_Bivar_SLP3-150-100-F
- D1: value LTST-C19HE1WT-H -> APFA3010LSEEZGKQBKC; footprint LED_SMD:LED_LiteOn_LTST-C19HE1WT -> LED_SMD:LED_Kingbright_APFA3010_3x1.5mm_Horizontal
- moved C31 2.29 mm to (164.8, 110.6), turned to 180 degrees
- moved D1 1.13 mm to (168.1, 111.4), turned to 90 degrees
Connections:
- D1 pad 2: Net-(D1-GK) -> +3V3
- D1 pad 3: Net-(D1-BK) -> Net-(D1-G)
- D1 pad 4: +3V3 -> Net-(D1-B)
- U5 pad 7: Net-(D1-GK) -> Net-(D1-G)
- U5 pad 8: Net-(D1-BK) -> Net-(D1-B)
Routing:
- net GND: track 11.3 -> 15.1 mm, vias 141 -> 140
- net Net-(D1-BK): track 3.77 -> 0.00 mm, vias 1 -> 0
- net Net-(D1-G): track 0.00 -> 3.62 mm, vias 0 -> 1
- net Net-(D1-B): track 0.00 -> 2.05 mm, vias 0 -> 1
- net Net-(D1-GK): track 2.01 -> 0.00 mm, vias 1 -> 0
- net Net-(D1-R): track 2.11 -> 3.99 mm
