File: hardware/pcb/kxusbc2.kicad_pcb (KiCad board)
At the start: 4 copper layers, 69 x 19 mm, 98 parts, among them J1 Conn_01x03, J2 UPDI, J3 Conn_01x03, J4 Conn_01x03, J5 GT-USB-7055AB, J6 Serial, J7 Conn_01x01, J8 Conn_01x01, Q1 CSD17581Q3A, Q2 CSD17581Q3A, Q3 CSD17581Q3A, Q4 CSD17581Q3A, Q5 CSD25402Q3A, SW1 SW_Push, U1 BQ25792RQMR, U2 ATtiny3226-M, U3 TLV9301xDCK, U4 RT9058-33GV, U5 LP5815DRLR, U7 FUSB302BMPX, Y1 32.768 kHz

Commit message: Move inductor slightly away from bottom edge
Parts:
- moved L1 0.20 mm to (137.1, 118.7)
Changed lines of the file:
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@@
 	(footprint "Inductor_SMD:L_APV_APH0630"
 		(layer "F.Cu")
-		(at 137.1 118.9 180)
+		(at 137.1 118.7 180)
 		(descr "Inductor, APV, APH0630, 6.8x6.6x2.8mm, (http://en.apvind.com/public/upload/20240408/996aafa961154ed753e4983e7eb80fa7.pdf), generated with kicad-footprint-generator gen_inductor.py")
 		(tags "molded power shielded")
@@
 	)
 	(via
-		(at 140.45 116.55)
+		(at 140.45 116.35)
 		(size 0.6)
 		(drill 0.4)
@@
 	)
 	(via
-		(at 133.65 115.7)
+		(at 133.65 115.6)
 		(size 0.6)
 		(drill 0.4)
@@
 	)
 	(via
-		(at 133.65 116.55)
+		(at 133.65 116.4)
 		(size 0.6)
 		(drill 0.4)
@@
 	)
 	(segment
-		(start 134.05 118.9)
-		(end 134.6 118.35)
+		(start 134.075 118.7)
+		(end 134.6 118.175)
 		(width 0.6)
 		(layer "F.Cu")
@@
 	)
 	(segment
-		(start 134.6 118.35)
+		(start 134.6 118.175)
 		(end 134.6 115.299997)
 		(width 0.6)
@@
 	)
 	(segment
+		(start 139.6 118.175)
+		(end 139.6 115.3)
+		(width 0.6)
+		(layer "F.Cu")
+		(net 29)
+	)
+	(segment
+		(start 140.125 118.7)
+		(end 139.6 118.175)
+		(width 0.6)
+		(layer "F.Cu")
+		(net 29)
+	)
+	(segment
 		(start 137.53375 111.25)
 		(end 137.53375 110.4)
@@
 		(layer "F.Cu")
 		(net 29)
-	)
-	(segment
-		(start 139.6 118.9)
-		(end 139.6 115.3)
-		(width 0.6)
-		(layer "F.Cu")
-		(net 29)

Commit message: Improve ground vias for SYS/PMID
Parts:
- moved TP1 1.27 mm to (135.2, 107.8)
Routing:
- net GND: vias 140 -> 141
Changed lines of the file:
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@@
 				(type "Bottom Silk Screen")
 			)
-			(copper_finish "HAL lead-free")
+			(copper_finish "ENIG")
 			(dielectric_constraints no)
 		)
@@
 	(footprint "TestPoint:TestPoint_Pad_2.5x2.5mm"
 		(layer "B.Cu")
-		(at 136.4 108)
+		(at 135.15 107.8)
 		(descr "SMD rectangular pad as test Point, square 2.5mm side length")
 		(tags "test point SMD pad rectangle square")
@@
 	)
 	(gr_text "GND"
-		(at 134.75 108.6 0)
+		(at 133.55 109.45 0)
 		(layer "B.SilkS")
 		(effects
@@
 	)
 	(segment
-		(start 137.08375 110.4)
-		(end 137.08375 109.26125)
+		(start 163.061 109.339)
+		(end 166.2775 109.339)
 		(width 0.2)
 		(layer "F.Cu")
@@
 	)
 	(segment
-		(start 163.061 109.339)
-		(end 166.2775 109.339)
+		(start 137.08375 110.4)
+		(end 137.08375 111.42094)
 		(width 0.2)
 		(layer "F.Cu")
@@
 	(segment
 		(start 137.08375 110.4)
-		(end 137.08375 111.42094)
+		(end 137.08375 109.315)
 		(width 0.2)
 		(layer "F.Cu")
@@
 	)
 	(segment
-		(start 136.6225 108.8)
-		(end 137.08375 109.26125)
+		(start 137.08375 109.26125)
+		(end 137.545 108.8)
 		(width 0.2)
 		(layer "F.Cu")
@@
 	)
 	(segment
-		(start 136.485 108.8)
+		(start 137.08375 109.26125)
 		(end 136.6225 108.8)
 		(width 0.2)
@@
 	)
 	(segment
-		(start 137.08375 109.26125)
-		(end 137.545 108.8)
+		(start 137.08375 109.315)
+		(end 137.08375 109.26125)
+		(width 0.2)
+		(layer "F.Cu")
+		(net 12)
+	)
+	(segment
+		(start 136.6225 108.8)
+		(end 136.485 108.8)
 		(width 0.2)
 		(layer "F.Cu")
@@
 	)
 	(via
+		(at 137.05 108.385)
+		(size 0.45)
+		(drill 0.3)
+		(layers "F.Cu" "B.Cu")
+		(free yes)
+		(net 12)
+	)
+	(via
 		(at 108.2 115.1)
 		(size 0.6)
@@
 	)
 	(via
-		(at 134.55 106.35)
-		(size 0.45)
-		(drill 0.3)
+		(at 139.25 124.15)
+		(size 0.6)
+		(drill 0.4)
 		(layers "F.Cu" "B.Cu")
 		(free yes)
@@
 	)
 	(via
-		(at 139.25 124.15)
-		(size 0.6)
-		(drill 0.4)
+		(at 137.08375 109.315)
+		(size 0.45)
+		(drill 0.3)
 		(layers "F.Cu" "B.Cu")
-		(free yes)
 		(net 12)
 	)

Commit message: Move some parts further away from bottom edge
Parts:
- moved R16 0.31 mm to (107.3, 121.2)
- moved C11 0.30 mm to (155.2, 123.5)
- moved R6 0.30 mm to (150.2, 121.3)
- moved R7 0.25 mm to (150.2, 123.2)
- moved R15 0.24 mm to (107.3, 123.2)
Routing:
- net GND: track 15.1 -> 16.0 mm, vias 141 -> 143
Changed lines of the file:
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@@
 	(footprint "Resistor_SMD:R_0402_1005Metric"
 		(layer "F.Cu")
-		(at 150.2 121.6 90)
+		(at 150.2 121.3 90)
 		(descr "Resistor SMD 0402 (1005 Metric), square (rectangular) end terminal, IPC-7351 nominal, (Body size source: IPC-SM-782 page 72, https://www.pcb-3d.com/wordpress/wp-content/uploads/ipc-sm-782a_amendment_1_and_2.pdf), generated with kicad-footprint-generator")
 		(tags "resistor")
@@
 	(footprint "Capacitor_SMD:C_0402_1005Metric"
 		(layer "F.Cu")
-		(at 155.15 123.85)
+		(at 155.15 123.55)
 		(descr "Capacitor SMD 0402 (1005 Metric), square (rectangular) end terminal, IPC-7351 nominal, (Body size source: IPC-SM-782 page 76, https://www.pcb-3d.com/wordpress/wp-content/uploads/ipc-sm-782a_amendment_1_and_2.pdf), generated with kicad-footprint-generator")
 		(tags "capacitor")
@@
 	(footprint "Resistor_SMD:R_0402_1005Metric"
 		(layer "F.Cu")
-		(at 107.29 121.51 -90)
+		(at 107.3 121.2 -90)
 		(descr "Resistor SMD 0402 (1005 Metric), square (rectangular) end terminal, IPC-7351 nominal, (Body size source: IPC-SM-782 page 72, https://www.pcb-3d.com/wordpress/wp-content/uploads/ipc-sm-782a_amendment_1_and_2.pdf), generated with kicad-footprint-generator")
 		(tags "resistor")
@@
 	(footprint "Resistor_SMD:R_0402_1005Metric"
 		(layer "F.Cu")
-		(at 150.2 123.5 -90)
+		(at 150.2 123.25 -90)
 		(descr "Resistor SMD 0402 (1005 Metric), square (rectangular) end terminal, IPC-7351 nominal, (Body size source: IPC-SM-782 page 72, https://www.pcb-3d.com/wordpress/wp-content/uploads/ipc-sm-782a_amendment_1_and_2.pdf), generated with kicad-footprint-generator")
 		(tags "resistor")
@@
 	(footprint "Resistor_SMD:R_0402_1005Metric"
 		(layer "F.Cu")
-		(at 107.29 123.39 -90)
+		(at 107.29 123.15 -90)
 		(descr "Resistor SMD 0402 (1005 Metric), square (rectangular) end terminal, IPC-7351 nominal, (Body size source: IPC-SM-782 page 72, https://www.pcb-3d.com/wordpress/wp-content/uploads/ipc-sm-782a_amendment_1_and_2.pdf), generated with kicad-footprint-generator")
 		(tags "resistor")
@@
 	)
 	(segment
+		(start 108.28 121)
+		(end 108.28 121.77)
+		(width 0.2)
+		(layer "F.Cu")
+		(net 12)
+	)
+	(segment
 		(start 117.25 110.6414)
 		(end 117.6 110.9914)
@@
 	)
 	(segment
+		(start 108.28 121.77)
+		(end 108.15 121.9)
+		(width 0.2)
+		(layer "F.Cu")
+		(net 12)
+	)
+	(segment
 		(start 165 112.35)
 		(end 165.45 112.35)
@@
 	)
 	(via
+		(at 149.35 124.25)
+		(size 0.45)
+		(drill 0.3)
+		(layers "F.Cu" "B.Cu")
+		(free yes)
+		(net 12)
+	)
+	(via
 		(at 112.05 119.365)
 		(size 0.45)
@@
 	)
 	(via
+		(at 152.65 124.2)
+		(size 0.45)
+		(drill 0.3)
+		(layers "F.Cu" "B.Cu")
+		(free yes)
+		(net 12)
+	)
+	(via
 		(at 158.4 117.55)
 		(size 0.6)
@@
 	)
 	(segment
-		(start 153.85 123.9)
-		(end 154.62 123.9)
-		(width 0.4)
-		(layer "F.Cu")
-		(net 26)
-	)
-	(segment
 		(start 107.29 118.8)
 		(end 107.29 117.99)
@@
 	)
 	(segment
-		(start 154.62 123.9)
-		(end 154.67 123.85)
-		(width 0.4)
-		(layer "F.Cu")
-		(net 26)
-	)
-	(segment
-		(start 150.2 122.11)
-		(end 150.2 122.99)
-		(width 0.2)
-		(layer "F.Cu")
-		(net 26)
-	)
-	(segment
-		(start 150.61 123.4)
-		(end 150.2 122.99)
-		(width 0.2)
-		(layer "F.Cu")
-		(net 26)
-	)
-	(segment
 		(start 108.63125 118.16875)
 		(end 108.725 118.2625)
@@
 	)
 	(segment
+		(start 153.55 123.6)
+		(end 154.62 123.6)
+		(width 0.4)
+		(layer "F.Cu")
+		(net 26)
+	)
+	(segment
 		(start 107.29 118.8)
 		(end 108 118.8)
@@
 	)
 	(segment
+		(start 154.62 123.6)
+		(end 154.67 123.55)
+		(width 0.4)
+		(layer "F.Cu")
+		(net 26)
+	)
+	(segment
 		(start 120.605473 115.4)
 		(end 121.5 115.4)
@@
 	)
 	(segment
-		(start 153.55 123.6)
-		(end 153.85 123.9)
-		(width 0.4)
+		(start 150.2 122.74)
+		(end 151.04 122.74)
+		(width 0.2)
+		(layer "F.Cu")
+		(net 26)
+	)
+	(segment
+		(start 151.04 122.74)
+		(end 151.7 123.4)
+		(width 0.2)
 		(layer "F.Cu")
 		(net 26)
@@
 	)
 	(segment
-		(start 151.7 123.4)
-		(end 150.61 123.4)
-		(width 0.2)
-		(layer "F.Cu")
-		(net 26)
-	)
-	(segment
 		(start 165.25 110.55)
 		(end 165.85 109.95)
@@
 		(net 26)
 	)
+	(segment
+		(start 150.2 121.81)
+		(end 150.2 122.74)
+		(width 0.2)
+		(layer "F.Cu")
+		(net 26)
+	)
 	(via
 		(at 153.55 123.6)
@@
 	)
 	(segment
+		(start 149.9 120.1)
+		(end 149.9 120.49)
+		(width 0.2)
+		(layer "F.Cu")
+		(net 41)
+	)
+	(segment
 		(start 137.68375 114.88375)
 		(end 137.8 115)
@@
 	)
 	(segment
-		(start 149.9 120.1)
-		(end 149.9 120.79)
+		(start 137.68375 114)
+		(end 137.68375 114.88375)
 		(width 0.2)
 		(layer "F.Cu")
@@
 	)
 	(segment
-		(start 137.68375 114)
-		(end 137.68375 114.88375)
+		(start 149.9 120.49)
+		(end 150.2 120.79)
 		(width 0.2)
 		(layer "F.Cu")
@@
 	)
 	(segment
-		(start 149.9 120.79)
-		(end 150.2 121.09)
-		(width 0.2)
-		(layer "F.Cu")
-		(net 41)
-	)
-	(segment
 		(start 167.8 111.4)
 		(end 167.8 110.7)
@@
 	)
 	(segment
-		(start 149.436 123.246)
-		(end 150.2 124.01)
-		(width 0.2)
-		(layer "F.Cu")
-		(net 42)
-	)
-	(segment
 		(start 110.4875 118.2625)
 		(end 111 118.775)
@@
 	)
 	(segment
-		(start 149.436 120.751)
-		(end 149.436 123.246)
+		(start 167.3 111.0895)
+		(end 167.3 110.7)
 		(width 0.2)
 		(layer "F.Cu")
@@
 	)
 	(segment
-		(start 167.3 111.0895)
-		(end 167.3 110.7)
+		(start 149.436 122.996)
+		(end 150.2 123.76)
 		(width 0.2)
 		(layer "F.Cu")
@@
 	)
 	(segment
-		(start 149.4 120.715)
-		(end 149.436 120.751)
+		(start 138.410003 114.895825)
+		(end 138.410003 115)
 		(width 0.2)
 		(layer "F.Cu")
@@
 	)
 	(segment
-		(start 138.410003 114.895825)
-		(end 138.410003 115)
+		(start 149.4 120.715)
+		(end 149.436 120.751)
 		(width 0.2)
 		(layer "F.Cu")
@@
 	)
 	(segment
+		(start 149.436 120.751)
+		(end 149.436 122.996)
+		(width 0.2)
+		(layer "F.Cu")
+		(net 42)
+	)
+	(segment
 		(start 111 118.775)
 		(end 111 119.2)
@@
 	)
 	(segment
-		(start 107.29 122.88)
-		(end 107.96 123.55)
+		(start 108.99 123.55)
+		(end 110.89 123.55)
 		(width 0.2)
 		(layer "F.Cu")
@@
 	)
 	(segment
-		(start 108.99 123.55)
-		(end 110.89 123.55)
+		(start 107.3 121.71)
+		(end 107.3 122.63)
 		(width 0.2)
 		(layer "F.Cu")
@@
 	)
 	(segment
-		(start 107.96 123.55)
+		(start 107.3 122.63)
+		(end 107.29 122.64)
+		(width 0.2)
+		(layer "F.Cu")
+		(net 53)
+	)
+	(segment
+		(start 108.2 123.55)
 		(end 108.99 123.55)
 		(width 0.2)
@@
 	)
 	(segment
-		(start 107.29 122.02)
-		(end 107.29 122.88)
+		(start 107.29 122.64)
+		(end 108.2 123.55)
 		(width 0.2)
 		(layer "F.Cu")
@@
 	)
 	(segment
-		(start 105.99 122.6)
-		(end 104.5 122.6)
+		(start 106.23 122.6)
+		(end 107.29 123.66)
 		(width 0.2)
 		(layer "F.Cu")
@@
 	)
 	(segment
-		(start 107.29 123.9)
-		(end 105.99 122.6)
+		(start 103.3 123.8)
+		(end 104.5 122.6)
 		(width 0.2)
 		(layer "F.Cu")
@@
 	(segment
 		(start 104.5 122.6)
-		(end 103.3 123.8)
+		(end 106.23 122.6)
 		(width 0.2)
 		(layer "F.Cu")

Commit message: SYS vias
Routing:
- net /Charger/SYS: track 12.9 -> 8.12 mm, vias 2 -> 8
Changed lines of the file:
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@@
-	)
-	(segment
-		(start 138.505 108.8)
-		(end 139.2 108.8)
-		(width 0.2)
-		(layer "F.Cu")
-		(net 31)
 	)
 	(segment
@@
 	)
 	(segment
-		(start 140.65 108.8)
-		(end 140.8 108.95)
-		(width 0.2)
-		(layer "F.Cu")
-		(net 31)
-	)
-	(segment
 		(start 137.98375 109.32125)
 		(end 138.505 108.8)
@@
 	)
 	(segment
-		(start 139.4 108.6)
-		(end 139.6 108.8)
-		(width 0.2)
-		(layer "F.Cu")
-		(net 31)
-	)
-	(segment
-		(start 139.2 108.8)
-		(end 139.4 108.6)
-		(width 0.2)
-		(layer "F.Cu")
-		(net 31)
-	)
-	(segment
 		(start 140.68375 108.775)
 		(end 140.45 108.775)
@@
 		(net 31)
 	)
-	(segment
-		(start 139.6 108.8)
-		(end 140.65 108.8)
-		(width 0.2)
-		(layer "F.Cu")
-		(net 31)
-	)
-	(via
-		(at 139.4 109.3)
-		(size 0.6)
+	(via
+		(at 141.789786 109.425846)
+		(size 0.45)
 		(drill 0.3)
 		(layers "F.Cu" "B.Cu")
@@
 	)
 	(via
-		(at 139.4 108.6)
-		(size 0.6)
-		(drill 0.3)
-		(layers "F.Cu" "B.Cu")
+		(at 139.2 109.45)
+		(size 0.45)
+		(drill 0.3)
+		(layers "F.Cu" "B.Cu")
+		(free yes)
+		(net 31)
+	)
+	(via
+		(at 139.2 108.95)
+		(size 0.45)
+		(drill 0.3)
+		(layers "F.Cu" "B.Cu")
+		(free yes)
+		(net 31)
+	)
+	(via
+		(at 139.2 108.45)
+		(size 0.45)
+		(drill 0.3)
+		(layers "F.Cu" "B.Cu")
+		(free yes)
+		(net 31)
+	)
+	(via
+		(at 139.75 108.95)
+		(size 0.45)
+		(drill 0.3)
+		(layers "F.Cu" "B.Cu")
+		(free yes)
+		(net 31)
+	)
+	(via
+		(at 139.75 109.45)
+		(size 0.45)
+		(drill 0.3)
+		(layers "F.Cu" "B.Cu")
+		(free yes)
+		(net 31)
+	)
+	(via
+		(at 141.8 108.45)
+		(size 0.45)
+		(drill 0.3)
+		(layers "F.Cu" "B.Cu")
+		(free yes)
+		(net 31)
+	)
+	(via
+		(at 139.75 108.45)
+		(size 0.45)
+		(drill 0.3)
+		(layers "F.Cu" "B.Cu")
+		(free yes)
 		(net 31)
 	)
@@
 	)
 	(segment
-		(start 139.75 108.95)
-		(end 139.4 108.6)
-		(width 0.4)
-		(layer "B.Cu")
-		(net 31)
-	)
-	(segment
-		(start 140.8 108.95)
-		(end 139.75 108.95)
-		(width 0.4)
-		(layer "B.Cu")
-		(net 31)
-	)
-	(segment
-		(start 139.4 109.3)
-		(end 139.4 108.6)
-		(width 0.4)
-		(layer "B.Cu")
-		(net 31)
-	)
-	(segment
 		(start 142.75 114.85)
 		(end 142.8 114.8)
@@
 	)
 	(segment
+		(start 137.8 109.8)
+		(end 129.7 109.8)
+		(width 0.2)
+		(layer "B.Cu")
+		(net 44)
+	)
+	(segment
+		(start 127.050748 112.449252)
+		(end 124.35 112.449252)
+		(width 0.2)
+		(layer "B.Cu")
+		(net 44)
+	)
+	(segment
+		(start 138.4 110.4)
+		(end 137.8 109.8)
+		(width 0.2)
+		(layer "B.Cu")
+		(net 44)
+	)
+	(segment
+		(start 140.4 111.1)
+		(end 139.7 110.4)
+		(width 0.2)
+		(layer "B.Cu")
+		(net 44)
+	)
+	(segment
+		(start 129.7 109.8)
+		(end 127.050748 112.449252)
+		(width 0.2)
+		(layer "B.Cu")
+		(net 44)
+	)
+	(segment
 		(start 140.4 111.65)
 		(end 140.4 111.1)
@@
 	)
 	(segment
-		(start 127.050748 112.449252)
-		(end 124.35 112.449252)
-		(width 0.2)
-		(layer "B.Cu")
-		(net 44)
-	)
-	(segment
-		(start 140.4 111.1)
-		(end 139.1 109.8)
-		(width 0.2)
-		(layer "B.Cu")
-		(net 44)
-	)
-	(segment
-		(start 129.7 109.8)
-		(end 127.050748 112.449252)
-		(width 0.2)
-		(layer "B.Cu")
-		(net 44)
-	)
-	(segment
-		(start 139.1 109.8)
-		(end 129.7 109.8)
-		(width 0.2)
-		(layer "B.Cu")
+		(start 139.7 110.4)
+		(end 138.4 110.4)
+		(width 0.2)
+		(layer "B.Cu")
