File: hardware/pcb/kxusbc2.kicad_pcb (KiCad board)
At the start: 4 copper layers, 69 x 19 mm, 98 parts, among them J1 Conn_01x03, J2 UPDI, J3 Conn_01x03, J4 Conn_01x03, J5 GT-USB-7055AB, J6 Serial, J7 Conn_01x01, J8 Conn_01x01, Q1 CSD17581Q3A, Q2 CSD17581Q3A, Q3 CSD17581Q3A, Q4 CSD17581Q3A, Q5 CSD25402Q3A, SW1 SW_Push, U1 BQ25792RQMR, U2 ATtiny3226-M, U3 TLV9301xDCK, U4 RT9058-33GV, U5 LP5815DRLR, U7 FUSB302BMPX, Y1 32.768 kHz

Commit message: Increase crystal load capacitors to 22p for more precise frequency pre-calibration
Parts:
- C32, C33: value 18p -> 22p
Other:
- board text added: "rev3a"
- board text removed: "rev3"
Changed lines of the file:
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@@
 			)
 		)
-		(property "Value" "18p"
+		(property "Value" "22p"
 			(at 0 1.16 0)
 			(layer "F.Fab")
@@
 			)
 		)
-		(property "LCSC" "C1549"
+		(property "LCSC" "C1555"
 			(at 0 0 0)
 			(layer "F.SilkS")
@@
 			)
 		)
-		(property "Value" "18p"
+		(property "Value" "22p"
 			(at 0 1.16 0)
 			(layer "F.Fab")
@@
 			)
 		)
-		(property "LCSC" "C1549"
+		(property "LCSC" "C1555"
 			(at 0 0 0)
 			(layer "F.SilkS")
@@
 		)
 	)
-	(gr_text "rev3"
+	(gr_text "rev3a"
 		(at 125.4 110.3 0)
 		(layer "B.SilkS")

Commit message: Offset LED 1 mm from edge for better mechanical protection
Parts:
- moved D1 1.00 mm to (167.1, 111.4)
Routing:
- net Net-(D1-R): track 3.99 -> 2.41 mm
- net Net-(D1-G): track 3.62 -> 4.98 mm
- net +3V3: track 94.6 -> 93.6 mm
Other:
- board text added: "rev4"
- board text removed: "rev3a"
