File: hardware/pcb/kxusbc2_btmon.kicad_sch (KiCad schematic)
At the start: 7 parts, among them U3 TLV9301xDCK

Commit message: Offset LED 1 mm from edge for better mechanical protection
Parts:
- R5: LCSC C11490 -> C138015
Changed lines of the file:
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@@
 		)
 		(instances
-			(project ""
+			(project "kxusbc2"
 				(path "/e3f9e6db-4c7d-434c-85a0-9bad2f7edcde/7c1acb59-0886-4fc3-b60c-8fe1068068b6"
 					(reference "#PWR018")
@@
 		)
 		(instances
-			(project ""
+			(project "kxusbc2"
 				(path "/e3f9e6db-4c7d-434c-85a0-9bad2f7edcde/7c1acb59-0886-4fc3-b60c-8fe1068068b6"
 					(reference "C15")
@@
 			)
 		)
-		(property "LCSC" "C11490"
+		(property "LCSC" "C138015"
 			(at 83.82 97.79 0)
 			(effects
@@
 		)
 		(instances
-			(project ""
+			(project "kxusbc2"
 				(path "/e3f9e6db-4c7d-434c-85a0-9bad2f7edcde/7c1acb59-0886-4fc3-b60c-8fe1068068b6"
 					(reference "R5")
@@
 		)
 		(instances
-			(project ""
+			(project "kxusbc2"
 				(path "/e3f9e6db-4c7d-434c-85a0-9bad2f7edcde/7c1acb59-0886-4fc3-b60c-8fe1068068b6"
 					(reference "U3")
